File: LaunchPad-Tester.sch (KiCad schematic (older format))
At the start: 10 parts, among them U1 CY8C9540A

Commit message: Renamed project to LaunchPad-Tester and coorected some typos.
Parts:
- H2: footprint (none) -> Socket_Strips:Socket_Strip_Straight_2x10_Pitch2.54mm
Changed lines of the file:
@@
 LIBS:contrib
 LIBS:valves
-LIBS:LauchpadTester
-LIBS:LaunchpadTester-cache
+LIBS:LaunchPad-Tester
+LIBS:LaunchPad-Tester-cache
 EELAYER 25 0
 EELAYER END
@@
 encoding utf-8
 Sheet 1 1
-Title ""
-Date ""
-Rev ""
+Title "LaunchPad-Tester"
+Date "2017-09-08"
+Rev "v1.0"
 Comp ""
 Comment1 ""
@@
 $EndComp
 $Comp
-L +3V3 #PWR1
+L +3V3 #PWR01
 U 1 1 599DAE5F
 P 1650 1450
-F 0 "#PWR1" H 1650 1300 50  0001 C CNN
+F 0 "#PWR01" H 1650 1300 50  0001 C CNN
 F 1 "+3V3" H 1650 1590 50  0000 C CNN
 F 2 "" H 1650 1450 50  0001 C CNN
@@
 	3050 2400 3525 2400
 $Comp
-L +3V3 #PWR7
+L +3V3 #PWR02
 U 1 1 599DB365
 P 4850 3600
-F 0 "#PWR7" H 4850 3450 50  0001 C CNN
+F 0 "#PWR02" H 4850 3450 50  0001 C CNN
 F 1 "+3V3" H 4850 3740 50  0000 C CNN
 F 2 "" H 4850 3600 50  0001 C CNN
@@
 	2875 6000 3000 6000
 $Comp
-L GND #PWR3
+L GND #PWR03
 U 1 1 599DB3C4
 P 2875 6175
-F 0 "#PWR3" H 2875 5925 50  0001 C CNN
+F 0 "#PWR03" H 2875 5925 50  0001 C CNN
 F 1 "GND" H 2875 6025 50  0000 C CNN
 F 2 "" H 2875 6175 50  0001 C CNN
@@
 	6000 2400 6500 2400
 $Comp
-L GND #PWR9
+L GND #PWR04
 U 1 1 599DD180
 P 6650 1500
-F 0 "#PWR9" H 6650 1250 50  0001 C CNN
+F 0 "#PWR04" H 6650 1250 50  0001 C CNN
 F 1 "GND" H 6650 1350 50  0000 C CNN
 F 2 "" H 6650 1500 50  0001 C CNN
@@
 	3050 1600 3650 1600
 $Comp
-L GND #PWR4
+L GND #PWR05
 U 1 1 599DD83B
 P 3650 1600
-F 0 "#PWR4" H 3650 1350 50  0001 C CNN
+F 0 "#PWR05" H 3650 1350 50  0001 C CNN
 F 1 "GND" H 3650 1450 50  0000 C CNN
 F 2 "" H 3650 1600 50  0001 C CNN
@@
 $EndComp
 $Comp
-L +3V3 #PWR5
+L +3V3 #PWR06
 U 1 1 599DE92E
 P 3850 3000
-F 0 "#PWR5" H 3850 2850 50  0001 C CNN
+F 0 "#PWR06" H 3850 2850 50  0001 C CNN
 F 1 "+3V3" H 3850 3140 50  0000 C CNN
 F 2 "" H 3850 3000 50  0001 C CNN
@@
 $EndComp
 $Comp
-L GND #PWR6
+L GND #PWR07
 U 1 1 599DE94A
 P 3850 3300
-F 0 "#PWR6" H 3850 3050 50  0001 C CNN
+F 0 "#PWR07" H 3850 3050 50  0001 C CNN
 F 1 "GND" H 3850 3150 50  0000 C CNN
 F 2 "" H 3850 3300 50  0001 C CNN
@@
 $EndComp
 $Comp
-L +3V3 #PWR2
+L +3V3 #PWR08
 U 1 1 599DECDF
 P 1875 5550
-F 0 "#PWR2" H 1875 5400 50  0001 C CNN
+F 0 "#PWR08" H 1875 5400 50  0001 C CNN
 F 1 "+3V3" H 1875 5690 50  0000 C CNN
 F 2 "" H 1875 5550 50  0001 C CNN
@@
 $EndComp
 $Comp
-L GND #PWR8
+L GND #PWR09
 U 1 1 599DF24B
 P 6300 5900
-F 0 "#PWR8" H 6300 5650 50  0001 C CNN
+F 0 "#PWR09" H 6300 5650 50  0001 C CNN
 F 1 "GND" H 6300 5750 50  0000 C CNN
 F 2 "" H 6300 5900 50  0001 C CNN
@@
 F 0 "H2" H 5050 2550 60  0000 C CNN
 F 1 "Header-J4-J2" H 5350 1350 60  0000 C CNN
-F 2 "" H 5150 1800 60  0001 C CNN
+F 2 "Socket_Strips:Socket_Strip_Straight_2x10_Pitch2.54mm" H 5150 1800 60  0001 C CNN
 F 3 "" H 5150 1800 60  0001 C CNN
 	1    5400 1950
